File: newProject/newProject.kicad_sch (KiCad schematic)
At the start: 32 parts, among them J1 Screw3, J10 Motor1 Output, J11 Motor2 Output, J12 xt30, J2 Screw3, J3 Screw3, J4 Screw3, J5 Screw3, J6 Conn_01x03_Pin, J7 Screw3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

Commit message: final update
Parts:
- removed J6: Conn_01x03_Pin, Connector_PinHeader_2.54mm:PinHeader_1x03_P2.54mm_Vertical, symbol Connector:Conn_01x03_Pin
- J10, J11: footprint JOEJOE:screw2 -> Connector_PinHeader_2.54mm:PinHeader_1x02_P2.54mm_Vertical
- J7: footprint Connector_JST:JST_EH_B3B-EH-A_1x03_P2.50mm_Vertical -> Connector_PinHeader_2.54mm:PinHeader_1x03_P2.54mm_Vertical
- PS1: footprint JOEJOE:convertor -> Battery:CONV_P78E05-1000
- SW2: footprint JOEJOE:realswitch -> Connector_PinHeader_2.54mm:PinHeader_1x03_P2.54mm_Vertical
- TB1: footprint JOEJOE:nano -> Module:Arduino_Nano
- U1: footprint JOEJOE:spoarkfun -> Module:MODULE_ROB-14450
Connections:
- net Servo is gone; now on net MOTOR1A: TB1.12 (D9)
- net MOTOR1A: no longer TB1.2 (D0/RX)
- net DIP1: no longer names the net of TB1.25 (A6)
- net DIP2: no longer names the net of TB1.26 (A7)
- no-connect marks 8 -> 10
Other:
- moved on the sheet: SW2A
