File: newProject/newProject.kicad_pcb (KiCad board)
At the start: 2 copper layers, 100 x 39 mm, 31 parts, among them J1 Screw3, J10 Motor1 Output, J11 Motor2 Output, J12 xt30, J2 Screw3, J3 Screw3, J4 Screw3, J5 Screw3, J7 Screw3, J8 Screw3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

Commit message: stuff
Parts:
- moved J9 6.14 mm to (88.5, 67.6)
- moved J8 2.00 mm to (168.3, 41.6)
- moved J7 1.50 mm to (86.5, 41.0)
Routing:
- net +5V: track 126.9 -> 134.7 mm
- net ST: track 24.6 -> 30.1 mm
- net LN2: track 73.1 -> 75.1 mm
- net LN1: track 43.5 -> 45.0 mm
Changed lines of the file:
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@@
 			(drillshape 0)
 			(scaleselection 1)
-			(outputdirectory "../../../../Desktop/robowrestling/")
+			(outputdirectory "../../../../Desktop/MagnoliaGerber/")
 		)
 	)
@@
 	(footprint "Connector_PinHeader_2.54mm:PinHeader_1x03_P2.54mm_Vertical"
 		(layer "F.Cu")
-		(at 88.5 61.42)
+		(at 88.5 67.56)
 		(descr "Through hole straight pin header, 1x03, 2.54mm pitch, single row")
 		(tags "Through hole pin header THT 1x03 2.54mm single row")
@@
 	(footprint "Connector_JST:JST_EH_B3B-EH-A_1x03_P2.50mm_Vertical"
 		(layer "F.Cu")
-		(at 166.3 41.5 -90)
+		(at 168.3 41.6 -90)
 		(descr "JST EH series connector, B3B-EH-A (http://www.jst-mfg.com/product/pdf/eng/eEH.pdf), generated with kicad-footprint-generator")
 		(tags "connector JST EH vertical")
@@
 	(footprint "Connector_PinHeader_2.54mm:PinHeader_1x03_P2.54mm_Vertical"
 		(layer "F.Cu")
-		(at 88 40.975)
+		(at 86.5 40.96)
 		(descr "Through hole straight pin header, 1x03, 2.54mm pitch, single row")
 		(tags "Through hole pin header THT 1x03 2.54mm single row")
@@
 	)
 	(segment
-		(start 86 60)
-		(end 86 64)
+		(start 89.55 50.5)
+		(end 92 52.95)
 		(width 0.2)
 		(layer "F.Cu")
@@
 	)
 	(segment
-		(start 89.55 50.5)
-		(end 92 52.95)
+		(start 92 54)
+		(end 86 60)
+		(width 0.2)
+		(layer "F.Cu")
+		(net 3)
+	)
+	(segment
+		(start 97.86 72.64)
+		(end 98.5 72)
+		(width 0.2)
+		(layer "F.Cu")
+		(net 3)
+	)
+	(segment
+		(start 86 70.14)
+		(end 88.5 72.64)
 		(width 0.2)
 		(layer "F.Cu")
@@
 	)
 	(segment
+		(start 88.0725 46.1275)
+		(end 87.985 46.04)
+		(width 0.2)
+		(layer "F.Cu")
+		(net 3)
+	)
+	(segment
 		(start 89.55 47.605)
-		(end 88 46.055)
+		(end 88.0725 46.1275)
 		(width 0.2)
 		(layer "F.Cu")
@@
 	)
 	(segment
-		(start 93 66.5)
-		(end 98.5 72)
+		(start 88.5 72.64)
+		(end 97.86 72.64)
 		(width 0.2)
 		(layer "F.Cu")
@@
 	)
 	(segment
-		(start 88.5 66.5)
-		(end 93 66.5)
+		(start 88.0725 46.1275)
+		(end 88 46.055)
+		(width 0.2)
+		(layer "F.Cu")
+		(net 3)
+	)
+	(segment
+		(start 87.985 46.04)
+		(end 86.5 46.04)
 		(width 0.2)
 		(layer "F.Cu")
@@
 	)
 	(segment
-		(start 89.55 50.5)
-		(end 89.55 47.605)
+		(start 86 60)
+		(end 86 70.14)
 		(width 0.2)
 		(layer "F.Cu")
@@
 	)
 	(segment
-		(start 92 54)
-		(end 86 60)
+		(start 89.55 50.5)
+		(end 89.55 47.605)
 		(width 0.2)
 		(layer "F.Cu")
@@
 		(net 3)
 	)
-	(segment
-		(start 86 64)
-		(end 88.5 66.5)
-		(width 0.2)
-		(layer "F.Cu")
-		(net 3)
-	)
 	(via
 		(at 133.250476 66.501)
@@
 	)
 	(segment
+		(start 166.4 46.6)
+		(end 168.3 46.6)
+		(width 0.2)
+		(layer "B.Cu")
+		(net 3)
+	)
+	(segment
 		(start 150.5 68)
 		(end 150.5 68.97)
@@
 	)
 	(segment
+		(start 166.3 46.5)
+		(end 166.4 46.6)
+		(width 0.2)
+		(layer "B.Cu")
+		(net 3)
+	)
+	(segment
 		(start 156 41.5)
 		(end 156.5 41.5)
@@
 	)
 	(segment
+		(start 96.601 62.612034)
+		(end 96.601 51.751057)
+		(width 0.2)
+		(layer "F.Cu")
+		(net 15)
+	)
+	(segment
 		(start 109.7 69)
 		(end 102.988966 69)
@@
 	)
 	(segment
-		(start 96.601 62.612034)
-		(end 96.601 51.751057)
+		(start 96.601 51.751057)
+		(end 89.200943 44.351)
 		(width 0.2)
 		(layer "F.Cu")
@@
 	)
 	(segment
-		(start 89.200943 44.351)
-		(end 89.151 44.351)
+		(start 102.988966 69)
+		(end 96.601 62.612034)
 		(width 0.2)
 		(layer "F.Cu")
@@
 	)
 	(segment
-		(start 89.151 44.351)
-		(end 89.151 42.126)
+		(start 89.151 42.126)
+		(end 87.985 40.96)
 		(width 0.2)
 		(layer "F.Cu")
@@
 	)
 	(segment
-		(start 96.601 51.751057)
-		(end 89.200943 44.351)
+		(start 89.151 44.351)
+		(end 89.151 42.126)
 		(width 0.2)
 		(layer "F.Cu")
@@
 	)
 	(segment
-		(start 111.46 67.24)
-		(end 109.7 69)
+		(start 89.200943 44.351)
+		(end 89.151 44.351)
 		(width 0.2)
 		(layer "F.Cu")
@@
 	)
 	(segment
-		(start 102.988966 69)
-		(end 96.601 62.612034)
+		(start 111.46 67.24)
+		(end 109.7 69)
 		(width 0.2)
 		(layer "F.Cu")
@@
 	)
 	(segment
-		(start 89.151 42.126)
-		(end 88 40.975)
+		(start 87.985 40.96)
+		(end 86.5 40.96)
 		(width 0.2)
 		(layer "F.Cu")
@@
 	)
 	(segment
+		(start 166.3 41.5)
+		(end 166.4 41.6)
+		(width 0.2)
+		(layer "F.Cu")
+		(net 16)
+	)
+	(segment
 		(start 114 67.24)
 		(end 115.339 65.901)
@@
 	)
 	(segment
+		(start 166.4 41.6)
+		(end 168.3 41.6)
+		(width 0.2)
+		(layer "F.Cu")
+		(net 16)
+	)
+	(segment
 		(start 167.5 49.45276)
 		(end 165.024 46.97676)
@@
 	)
 	(segment
-		(start 91.08 61.42)
+		(start 88.5 67.56)
+		(end 88.5 64)
+		(width 0.2)
+		(layer "F.Cu")
+		(net 17)
+	)
+	(segment
+		(start 88.5 64)
+		(end 91.7 60.8)
+		(width 0.2)
+		(layer "F.Cu")
+		(net 17)
+	)
+	(segment
+		(start 91.7 60.8)
 		(end 96 56.5)
 		(width 0.2)
@@
 	)
 	(segment
-		(start 88.5 61.42)
-		(end 91.08 61.42)
+		(start 91.08 61.42)
+		(end 91.7 60.8)
 		(width 0.2)
 		(layer "F.Cu")
